File: pcb-r1/Power.sch (KiCad schematic (older format))
At the start: 22 parts, among them P301 USB-MICRO-B, P302 CONN_01X02, U301 FT232RQ, U302 MCP1700T-3302E

Commit message: Started preliminary layout of the parts
Parts:
- C301, C302, C303, C304: footprint (none) -> Capacitors_SMD:C_0805
- C305, C306: footprint Capacitors_SMD:C_0805 -> Capacitors_SMD:C_1210
- D301, D302: footprint (none) -> Diodes_SMD:SMA_Standard
- D303, D304: footprint (none) -> LEDs:LED-0805
- L301: footprint (none) -> Inductors_NEOSID:Neosid_Inductor_SM1206
- P301: footprint (none) -> CentralCommand:USB_Micro_B
- P302: footprint (none) -> Pin_Headers:Pin_Header_Straight_1x02
- R301, R302, R303, R304, R305, R306, R307: footprint (none) -> Resistors_SMD:R_0805
- U301: footprint (none) -> Housings_DFN_QFN:QFN-32-1EP_5x5mm_Pitch0.5mm
- U302: footprint Housings_SOT-23_SOT-143_TSOT-6:SOT-23 -> TO_SOT_Packages_SMD:SOT-23
Changed lines of the file:
@@
 F 0 "U302" H 6550 2800 60  0000 C CNN
 F 1 "MCP1700T-3302E" H 6050 3200 60  0000 C CNN
-F 2 "Housings_SOT-23_SOT-143_TSOT-6:SOT-23" H 5950 3300 60  0001 C CNN
+F 2 "TO_SOT_Packages_SMD:SOT-23" H 5950 3300 60  0001 C CNN
 F 3 "" H 5950 3300 60  0000 C CNN
 F 4 "http://parts.io/detail/1370896/MCP1700T-3302E%2FTT" H 6050 3150 60  0001 C CNN "link"
@@
 F 0 "C306" H 7125 3350 50  0000 L CNN
 F 1 "10μF" H 7125 3150 50  0000 L CNN
-F 2 "Capacitors_SMD:C_0805" H 7138 3100 30  0001 C CNN
+F 2 "Capacitors_SMD:C_1210" H 7138 3100 30  0001 C CNN
 F 3 "" H 7100 3250 60  0000 C CNN
 	1    7100 3250
@@
 F 0 "C305" H 5225 3400 50  0000 L CNN
 F 1 "10μF" H 5225 3200 50  0000 L CNN
-F 2 "Capacitors_SMD:C_0805" H 5238 3150 30  0001 C CNN
+F 2 "Capacitors_SMD:C_1210" H 5238 3150 30  0001 C CNN
 F 3 "" H 5200 3300 60  0000 C CNN
 	1    5200 3300
@@
 F 0 "P302" H 3300 3150 50  0000 C CNN
 F 1 "CONN_01X02" V 3400 3000 50  0000 C CNN
-F 2 "" H 3300 3000 60  0001 C CNN
+F 2 "Pin_Headers:Pin_Header_Straight_1x02" H 3300 3000 60  0001 C CNN
 F 3 "" H 3300 3000 60  0000 C CNN
 	1    3300 3000
@@
 F 0 "U301" H 5950 5350 60  0000 C CNN
 F 1 "FT232RQ" H 5950 5500 60  0000 C CNN
-F 2 "" H 5650 6000 60  0001 C CNN
+F 2 "Housings_DFN_QFN:QFN-32-1EP_5x5mm_Pitch0.5mm" H 5650 6000 60  0001 C CNN
 F 3 "http://www.ftdichip.com/Support/Documents/DataSheets/ICs/DS_FT232R.pdf" H 5650 6000 60  0001 C CNN
 	1    5950 5400
@@
 F 0 "P301" H 2350 5050 50  0000 C CNN
 F 1 "USB-MICRO-B" H 2500 4350 50  0000 C CNN
-F 2 "" H 2650 4600 50  0001 C CNN
+F 2 "CentralCommand:USB_Micro_B" H 2650 4600 50  0001 C CNN
 F 3 "" H 2650 4600 50  0000 C CNN
 	1    2650 4700
@@
 F 0 "L301" H 3800 4600 50  0000 C CNN
 F 1 "FERRITE" H 3800 4450 50  0000 C CNN
-F 2 "" H 3800 4500 60  0001 C CNN
+F 2 "Inductors_NEOSID:Neosid_Inductor_SM1206" H 3800 4500 60  0001 C CNN
 F 3 "" H 3800 4500 60  0000 C CNN
 	1    3800 4500
@@
 F 0 "C301" H 3475 5300 50  0000 L CNN
 F 1 "0.01μF" H 3475 5100 50  0000 L CNN
-F 2 "" H 3488 5050 30  0001 C CNN
+F 2 "Capacitors_SMD:C_0805" H 3488 5050 30  0001 C CNN
 F 3 "" H 3450 5200 60  0000 C CNN
 	1    3450 5200
@@
 F 0 "D301" H 3800 3050 50  0000 C CNN
 F 1 "D_Schottky" H 3800 2850 50  0000 C CNN
-F 2 "" H 3800 2950 60  0001 C CNN
+F 2 "Diodes_SMD:SMA_Standard" H 3800 2950 60  0001 C CNN
 F 3 "" H 3800 2950 60  0000 C CNN
 	1    3800 2950
@@
 F 0 "D302" H 4100 4250 50  0000 C CNN
 F 1 "D_Schottky" H 4100 4050 50  0000 C CNN
-F 2 "" H 4100 4150 60  0001 C CNN
+F 2 "Diodes_SMD:SMA_Standard" H 4100 4150 60  0001 C CNN
 F 3 "" H 4100 4150 60  0000 C CNN
 	1    4100 4150
@@
 F 0 "C302" H 4075 6750 50  0000 L CNN
 F 1 "0.1μF" H 4075 6550 50  0000 L CNN
-F 2 "" H 4088 6500 30  0001 C CNN
+F 2 "Capacitors_SMD:C_0805" H 4088 6500 30  0001 C CNN
 F 3 "" H 4050 6650 60  0000 C CNN
 	1    4050 6650
@@
 F 0 "C303" H 4425 6750 50  0000 L CNN
 F 1 "4.7μF" H 4425 6550 50  0000 L CNN
-F 2 "" H 4438 6500 30  0001 C CNN
+F 2 "Capacitors_SMD:C_0805" H 4438 6500 30  0001 C CNN
 F 3 "" H 4400 6650 60  0000 C CNN
 	1    4400 6650
@@
 F 0 "C304" H 4925 6750 50  0000 L CNN
 F 1 "0.1μF" H 4925 6550 50  0000 L CNN
-F 2 "" H 4938 6500 30  0001 C CNN
+F 2 "Capacitors_SMD:C_0805" H 4938 6500 30  0001 C CNN
 F 3 "" H 4900 6650 60  0000 C CNN
 	1    4900 6650
@@
 F 0 "R301" V 5030 5800 50  0000 C CNN
 F 1 "0Ω" V 4950 5800 50  0000 C CNN
-F 2 "" V 4880 5800 30  0001 C CNN
+F 2 "Resistors_SMD:R_0805" V 4880 5800 30  0001 C CNN
 F 3 "" H 4950 5800 30  0000 C CNN
 	1    4950 5800
@@
 F 0 "R306" V 8280 4900 50  0000 C CNN
 F 1 "270Ω" V 8200 4900 50  0000 C CNN
-F 2 "" V 8130 4900 30  0001 C CNN
+F 2 "Resistors_SMD:R_0805" V 8130 4900 30  0001 C CNN
 F 3 "" H 8200 4900 30  0000 C CNN
 	1    8200 4900
@@
 F 0 "D303" H 8200 5500 50  0000 C CNN
 F 1 "LED" H 8200 5300 50  0000 C CNN
-F 2 "" H 8200 5400 60  0001 C CNN
+F 2 "LEDs:LED-0805" H 8200 5400 60  0001 C CNN
 F 3 "" H 8200 5400 60  0000 C CNN
 	1    8200 5400
@@
 F 0 "R307" V 8730 4900 50  0000 C CNN
 F 1 "270Ω" V 8650 4900 50  0000 C CNN
-F 2 "" V 8580 4900 30  0001 C CNN
+F 2 "Resistors_SMD:R_0805" V 8580 4900 30  0001 C CNN
 F 3 "" H 8650 4900 30  0000 C CNN
 	1    8650 4900
@@
 F 0 "D304" H 8650 5500 50  0000 C CNN
 F 1 "LED" H 8650 5300 50  0000 C CNN
-F 2 "" H 8650 5400 60  0001 C CNN
+F 2 "LEDs:LED-0805" H 8650 5400 60  0001 C CNN
 F 3 "" H 8650 5400 60  0000 C CNN
 	1    8650 5400
@@
 F 0 "R304" V 7080 4800 50  0000 C CNN
 F 1 "NOPE" V 7000 4800 50  0000 C CNN
-F 2 "" V 6930 4800 30  0001 C CNN
+F 2 "Resistors_SMD:R_0805" V 6930 4800 30  0001 C CNN
 F 3 "" H 7000 4800 30  0000 C CNN
 	1    7000 4800
@@
 F 0 "R305" V 7080 4950 50  0000 C CNN
 F 1 "NOPE" V 7000 4950 50  0000 C CNN
-F 2 "" V 6930 4950 30  0001 C CNN
+F 2 "Resistors_SMD:R_0805" V 6930 4950 30  0001 C CNN
 F 3 "" H 7000 4950 30  0000 C CNN
 	1    7000 4950
@@
 F 0 "R302" V 7080 4500 50  0000 C CNN
 F 1 "0Ω" V 7000 4500 50  0000 C CNN
-F 2 "" V 6930 4500 30  0001 C CNN
+F 2 "Resistors_SMD:R_0805" V 6930 4500 30  0001 C CNN
 F 3 "" H 7000 4500 30  0000 C CNN
 	1    7000 4500
@@
 F 0 "R303" V 7080 4650 50  0000 C CNN
 F 1 "0Ω" V 7000 4650 50  0000 C CNN
-F 2 "" V 6930 4650 30  0001 C CNN
+F 2 "Resistors_SMD:R_0805" V 6930 4650 30  0001 C CNN
 F 3 "" H 7000 4650 30  0000 C CNN
 	1    7000 4650

Commit message: Intermediate save of the layout
Parts:
- P302: value CONN_01X02 -> ALT PWR
Connections:
- net labels added: VCCIO
- wire segments 75 -> 76
- no-connect marks 0 -> 16
Changed lines of the file:
@@
 $EndComp
 $Comp
-L GND #PWR010
+L GND #PWR011
 U 1 1 5657EDD1
 P 5800 4050
-F 0 "#PWR010" H 5800 3800 50  0001 C CNN
+F 0 "#PWR011" H 5800 3800 50  0001 C CNN
 F 1 "GND" H 5800 3900 50  0000 C CNN
 F 2 "" H 5800 4050 60  0000 C CNN
@@
 P 3300 3000
 F 0 "P302" H 3300 3150 50  0000 C CNN
-F 1 "CONN_01X02" V 3400 3000 50  0000 C CNN
+F 1 "ALT PWR" H 3300 2800 50  0000 C CNN
 F 2 "Pin_Headers:Pin_Header_Straight_1x02" H 3300 3000 60  0001 C CNN
 F 3 "" H 3300 3000 60  0000 C CNN
@@
 $EndComp
 $Comp
-L GND #PWR011
+L GND #PWR012
 U 1 1 5657F45C
 P 3600 3350
-F 0 "#PWR011" H 3600 3100 50  0001 C CNN
+F 0 "#PWR012" H 3600 3100 50  0001 C CNN
 F 1 "GND" H 3600 3200 50  0000 C CNN
 F 2 "" H 3600 3350 60  0000 C CNN
@@
 $EndComp
 $Comp
-L GND #PWR012
+L GND #PWR013
 U 1 1 565817D5
 P 3200 5600
-F 0 "#PWR012" H 3200 5350 50  0001 C CNN
+F 0 "#PWR013" H 3200 5350 50  0001 C CNN
 F 1 "GND" H 3200 5450 50  0000 C CNN
 F 2 "" H 3200 5600 60  0000 C CNN
@@
 $EndComp
 $Comp
-L GND #PWR013
+L GND #PWR014
 U 1 1 5659E477
 P 4250 7250
-F 0 "#PWR013" H 4250 7000 50  0001 C CNN
+F 0 "#PWR014" H 4250 7000 50  0001 C CNN
 F 1 "GND" H 4250 7100 50  0000 C CNN
 F 2 "" H 4250 7250 60  0000 C CNN
@@
 	1    0    0    -1
 $EndComp
-Text GLabel 4700 5800 0    60   Input ~ 0
-NRST
 $Comp
 L R R301
@@
 $EndComp
 $Comp
-L GND #PWR014
+L GND #PWR015
 U 1 1 5659F562
-P 5550 7150
-F 0 "#PWR014" H 5550 6900 50  0001 C CNN
-F 1 "GND" H 5550 7000 50  0000 C CNN
-F 2 "" H 5550 7150 60  0000 C CNN
-F 3 "" H 5550 7150 60  0000 C CNN
-	1    5550 7150
+P 5500 7050
+F 0 "#PWR015" H 5500 6800 50  0001 C CNN
+F 1 "GND" H 5500 6900 50  0000 C CNN
+F 2 "" H 5500 7050 60  0000 C CNN
+F 3 "" H 5500 7050 60  0000 C CNN
+	1    5500 7050
 	1    0    0    -1
 $EndComp
@@
 	5100 5800 5200 5800
 Wire Wire Line
-	5550 6900 5550 7150
-Wire Wire Line
-	5550 7000 6350 7000
-Wire Wire Line
-	6350 7000 6350 6900
-Wire Wire Line
-	6150 6900 6150 7000
-Connection ~ 6150 7000
-Wire Wire Line
-	5950 6900 5950 7000
-Connection ~ 5950 7000
-Wire Wire Line
-	5750 6900 5750 7000
-Connection ~ 5750 7000
-Connection ~ 5550 7000
-Wire Wire Line
 	8200 5050 8200 5200
 Wire Wire Line
@@
 	7300 4950 7150 4950
 $Comp
-L GND #PWR015
+L GND #PWR016
 U 1 1 565A0941
 P 7300 5100
-F 0 "#PWR015" H 7300 4850 50  0001 C CNN
+F 0 "#PWR016" H 7300 4850 50  0001 C CNN
 F 1 "GND" H 7300 4950 50  0000 C CNN
 F 2 "" H 7300 5100 60  0000 C CNN
@@
 GND
 Connection ~ 7100 3800
+Wire Wire Line
+	5500 6900 5500 7050
+Wire Wire Line
+	5500 6950 6450 6950
+Wire Wire Line
+	5800 6950 5800 6900
+Connection ~ 5500 6950
+Wire Wire Line
+	5900 6950 5900 6900
+Connection ~ 5800 6950
+Wire Wire Line
+	6000 6950 6000 6900
+Connection ~ 5900 6950
+Wire Wire Line
+	6100 6950 6100 6900
+Connection ~ 6000 6950
+Wire Wire Line
+	6450 6950 6450 6900
+Connection ~ 6100 6950
+Text Label 5250 4300 0    60   ~ 0
+VCCIO
+Text HLabel 4700 5800 0    60   Input ~ 0
+NRST
+NoConn ~ 3150 4800
+NoConn ~ 5200 5100
+NoConn ~ 5200 5200
+NoConn ~ 5200 5350
+NoConn ~ 5200 5500
+NoConn ~ 5200 5650
+NoConn ~ 5200 5950
+NoConn ~ 6700 5100
+NoConn ~ 6700 5250
+NoConn ~ 6700 5400
+NoConn ~ 6700 5550
+NoConn ~ 6700 6000
+NoConn ~ 6700 6150
+NoConn ~ 6700 6300
+NoConn ~ 5200 6250
+NoConn ~ 5200 6100
 $EndSCHEMATC

Commit message: Final draft layout. Published to build log as V01
Parts:
- D303: value LED -> Tx LED
- D304: value LED -> Rx LED
Changed lines of the file:
@@
 P 8200 5400
 F 0 "D303" H 8200 5500 50  0000 C CNN
-F 1 "LED" H 8200 5300 50  0000 C CNN
+F 1 "Tx LED" H 8200 5300 50  0000 C CNN
 F 2 "LEDs:LED-0805" H 8200 5400 60  0001 C CNN
 F 3 "" H 8200 5400 60  0000 C CNN
@@
 P 8650 5400
 F 0 "D304" H 8650 5500 50  0000 C CNN
-F 1 "LED" H 8650 5300 50  0000 C CNN
+F 1 "Rx LED" H 8650 5300 50  0000 C CNN
 F 2 "LEDs:LED-0805" H 8650 5400 60  0001 C CNN
 F 3 "" H 8650 5400 60  0000 C CNN
