File: pcb-r1/Power.sch (KiCad schematic (older format))
At the start: 22 parts, among them P301 USB-MICRO-B, P302 ALT PWR, U301 FT232RQ, U302 MCP1700T-3302E

Commit message: Updated the L301 to a 1206 part rather than 0603
Parts:
- L301: DigiKeyPN 732-4661-1-ND -> 490-5989-1-ND; MPN 742792605 -> BLM31PG330SN1L
Changed lines of the file:
@@
 F 2 "Inductors_NEOSID:Neosid_Inductor_SM1206" H 3800 4500 60  0001 C CNN
 F 3 "" H 3800 4500 60  0000 C CNN
-F 4 "742792605" H 3800 4500 60  0001 C CNN "MPN"
+F 4 "BLM31PG330SN1L" H 3800 4500 60  0001 C CNN "MPN"
 F 5 "Value" H 3800 4500 60  0001 C CNN "ConradPN"
 F 6 "Value" H 3800 4500 60  0000 C CNN "Label"
-F 7 "732-4661-1-ND" H 3800 4500 60  0001 C CNN "DigiKeyPN"
+F 7 "490-5989-1-ND" H 3800 4500 60  0001 C CNN "DigiKeyPN"
 	1    3800 4500
 	1    0    0    -1
